Commit message: UR10e working

File: rtb-data/rtbdata/xacro/ur_e_description/urdf/ur10_macro.xacro (robot description, xacro)
@@ -3,7 +3,7 @@
   <!--
     Convenience wrapper for the 'ur_robot' macro which provides default values
-    for the various "parameters files" parameters for a UR3.
+    for the various "parameters files" parameters for a UR10.
     This file can be used when composing a more complex scene with one or more
-    UR3 robots.
+    UR10 robots.
     While the generic 'ur_robot' macro could also be used, it would require
     the user to provide values for all parameters, as that macro does not set
@@ -17,10 +17,10 @@
           real robot.
   -->
-  <xacro:macro name="ur3_robot" params="
+  <xacro:macro name="ur10_robot" params="
    prefix
-   joint_limits_parameters_file:='$(find ur_description)/config/ur3/joint_limits.yaml'
-   kinematics_parameters_file:='$(find ur_description)/config/ur3/default_kinematics.yaml'
-   physical_parameters_file:='$(find ur_description)/config/ur3/physical_parameters.yaml'
-   visual_parameters_file:='$(find ur_description)/config/ur3/visual_parameters.yaml'
+   joint_limits_parameters_file:='$(find ur_description)/config/ur10/joint_limits.yaml'
+   kinematics_parameters_file:='$(find ur_description)/config/ur10/default_kinematics.yaml'
+   physical_parameters_file:='$(find ur_description)/config/ur10/physical_parameters.yaml'
+   visual_parameters_file:='$(find ur_description)/config/ur10/visual_parameters.yaml'
    transmission_hw_interface:=hardware_interface/PositionJointInterface
    safety_limits:=false
@@ -28,5 +28,5 @@
    safety_k_position:=20"
   >
-    <xacro:include filename="$(find ur_description)/urdf/inc/ur_macro.xacro"/>
+    <xacro:include filename="$(find ur_description)/urdf/ur_macro.xacro"/>
     <xacro:ur_robot
       prefix="${prefix}"

File: rtb-data/rtbdata/xacro/ur_e_description/urdf/ur10e.xacro (robot description, xacro)
@@ -14,5 +14,5 @@
     Refer to 'inc/ur_macro.xacro' for more information.
   -->
-  <xacro:include filename="$(find ur_description)/urdf/inc/ur10e_macro.xacro"/>
+  <xacro:include filename="$(find ur_description)/urdf/ur10e_macro.xacro"/>
   <xacro:ur10e_robot prefix="" />
 </robot>

File: rtb-data/rtbdata/xacro/ur_e_description/urdf/ur10e_macro.xacro (robot description, xacro)
@@ -3,7 +3,7 @@
   <!--
     Convenience wrapper for the 'ur_robot' macro which provides default values
-    for the various "parameters files" parameters for a UR5e.
+    for the various "parameters files" parameters for a UR10e.
     This file can be used when composing a more complex scene with one or more
-    UR5e robots.
+    UR10e robots.
     While the generic 'ur_robot' macro could also be used, it would require
     the user to provide values for all parameters, as that macro does not set
@@ -17,10 +17,10 @@
           real robot.
   -->
-  <xacro:macro name="ur5e_robot" params="
+  <xacro:macro name="ur10e_robot" params="
    prefix
-   joint_limits_parameters_file:='$(find ur_description)/config/ur5e/joint_limits.yaml'
-   kinematics_parameters_file:='$(find ur_description)/config/ur5e/default_kinematics.yaml'
-   physical_parameters_file:='$(find ur_description)/config/ur5e/physical_parameters.yaml'
-   visual_parameters_file:='$(find ur_description)/config/ur5e/visual_parameters.yaml'
+   joint_limits_parameters_file:='$(find ur_description)/config/ur10e/joint_limits.yaml'
+   kinematics_parameters_file:='$(find ur_description)/config/ur10e/default_kinematics.yaml'
+   physical_parameters_file:='$(find ur_description)/config/ur10e/physical_parameters.yaml'
+   visual_parameters_file:='$(find ur_description)/config/ur10e/visual_parameters.yaml'
    transmission_hw_interface:=hardware_interface/PositionJointInterface
    safety_limits:=false
@@ -28,5 +28,5 @@
    safety_k_position:=20"
   >
-    <xacro:include filename="$(find ur_description)/urdf/inc/ur_macro.xacro"/>
+    <xacro:include filename="$(find ur_description)/urdf/ur_macro.xacro"/>
     <xacro:ur_robot
       prefix="${prefix}"

File: rtb-data/rtbdata/xacro/ur_e_description/urdf/ur16e_macro.xacro (robot description, xacro)
@@ -3,7 +3,7 @@
   <!--
     Convenience wrapper for the 'ur_robot' macro which provides default values
-    for the various "parameters files" parameters for a UR10e.
+    for the various "parameters files" parameters for a UR16e.
     This file can be used when composing a more complex scene with one or more
-    UR10e robots.
+    UR16e robots.
     While the generic 'ur_robot' macro could also be used, it would require
     the user to provide values for all parameters, as that macro does not set
@@ -17,10 +17,10 @@
           real robot.
   -->
-  <xacro:macro name="ur10e_robot" params="
+  <xacro:macro name="ur16e_robot" params="
    prefix
-   joint_limits_parameters_file:='$(find ur_description)/config/ur10e/joint_limits.yaml'
-   kinematics_parameters_file:='$(find ur_description)/config/ur10e/default_kinematics.yaml'
-   physical_parameters_file:='$(find ur_description)/config/ur10e/physical_parameters.yaml'
-   visual_parameters_file:='$(find ur_description)/config/ur10e/visual_parameters.yaml'
+   joint_limits_parameters_file:='$(find ur_description)/config/ur16e/joint_limits.yaml'
+   kinematics_parameters_file:='$(find ur_description)/config/ur16e/default_kinematics.yaml'
+   physical_parameters_file:='$(find ur_description)/config/ur16e/physical_parameters.yaml'
+   visual_parameters_file:='$(find ur_description)/config/ur16e/visual_parameters.yaml'
    transmission_hw_interface:=hardware_interface/PositionJointInterface
    safety_limits:=false
@@ -28,5 +28,5 @@
    safety_k_position:=20"
   >
-    <xacro:include filename="$(find ur_description)/urdf/inc/ur_macro.xacro"/>
+    <xacro:include filename="$(find ur_description)/urdf/ur_macro.xacro"/>
     <xacro:ur_robot
       prefix="${prefix}"

File: rtb-data/rtbdata/xacro/ur_e_description/urdf/ur20_macro.xacro (robot description, xacro)
@@ -3,7 +3,7 @@
   <!--
     Convenience wrapper for the 'ur_robot' macro which provides default values
-    for the various "parameters files" parameters for a UR3e.
+    for the various "parameters files" parameters for a ur20.
     This file can be used when composing a more complex scene with one or more
-    UR3e robots.
+    ur20 robots.
     While the generic 'ur_robot' macro could also be used, it would require
     the user to provide values for all parameters, as that macro does not set
@@ -17,10 +17,10 @@
           real robot.
   -->
-  <xacro:macro name="ur3e_robot" params="
+  <xacro:macro name="ur20_robot" params="
    prefix
-   joint_limits_parameters_file:='$(find ur_description)/config/ur3e/joint_limits.yaml'
-   kinematics_parameters_file:='$(find ur_description)/config/ur3e/default_kinematics.yaml'
-   physical_parameters_file:='$(find ur_description)/config/ur3e/physical_parameters.yaml'
-   visual_parameters_file:='$(find ur_description)/config/ur3e/visual_parameters.yaml'
+   joint_limits_parameters_file:='$(find ur_description)/config/ur20/joint_limits.yaml'
+   kinematics_parameters_file:='$(find ur_description)/config/ur20/default_kinematics.yaml'
+   physical_parameters_file:='$(find ur_description)/config/ur20/physical_parameters.yaml'
+   visual_parameters_file:='$(find ur_description)/config/ur20/visual_parameters.yaml'
    transmission_hw_interface:=hardware_interface/PositionJointInterface
    safety_limits:=false
@@ -28,5 +28,5 @@
    safety_k_position:=20"
   >
-    <xacro:include filename="$(find ur_description)/urdf/inc/ur_macro.xacro"/>
+    <xacro:include filename="$(find ur_description)/urdf/ur_macro.xacro"/>
     <xacro:ur_robot
       prefix="${prefix}"

File: rtb-data/rtbdata/xacro/ur_e_description/urdf/ur30.xacro (robot description, xacro)
@@ -14,5 +14,5 @@
     Refer to 'inc/ur_macro.xacro' for more information.
   -->
-  <xacro:include filename="$(find ur_description)/urdf/inc/ur30_macro.xacro"/>
+  <xacro:include filename="$(find ur_description)/urdf/ur30_macro.xacro"/>
   <xacro:ur30_robot prefix="" />
 </robot>

File: rtb-data/rtbdata/xacro/ur_e_description/urdf/ur30_macro.xacro (robot description, xacro)
@@ -3,7 +3,7 @@
   <!--
     Convenience wrapper for the 'ur_robot' macro which provides default values
-    for the various "parameters files" parameters for a UR10.
+    for the various "parameters files" parameters for a ur30.
     This file can be used when composing a more complex scene with one or more
-    UR10 robots.
+    ur30 robots.
     While the generic 'ur_robot' macro could also be used, it would require
     the user to provide values for all parameters, as that macro does not set
@@ -17,10 +17,10 @@
           real robot.
   -->
-  <xacro:macro name="ur10_robot" params="
+  <xacro:macro name="ur30_robot" params="
    prefix
-   joint_limits_parameters_file:='$(find ur_description)/config/ur10/joint_limits.yaml'
-   kinematics_parameters_file:='$(find ur_description)/config/ur10/default_kinematics.yaml'
-   physical_parameters_file:='$(find ur_description)/config/ur10/physical_parameters.yaml'
-   visual_parameters_file:='$(find ur_description)/config/ur10/visual_parameters.yaml'
+   joint_limits_parameters_file:='$(find ur_description)/config/ur30/joint_limits.yaml'
+   kinematics_parameters_file:='$(find ur_description)/config/ur30/default_kinematics.yaml'
+   physical_parameters_file:='$(find ur_description)/config/ur30/physical_parameters.yaml'
+   visual_parameters_file:='$(find ur_description)/config/ur30/visual_parameters.yaml'
    transmission_hw_interface:=hardware_interface/PositionJointInterface
    safety_limits:=false
@@ -28,5 +28,5 @@
    safety_k_position:=20"
   >
-    <xacro:include filename="$(find ur_description)/urdf/inc/ur_macro.xacro"/>
+    <xacro:include filename="$(find ur_description)/urdf/ur_macro.xacro"/>
     <xacro:ur_robot
       prefix="${prefix}"

File: rtb-data/rtbdata/xacro/ur_e_description/urdf/ur3_macro.xacro (robot description, xacro)
@@ -3,7 +3,7 @@
   <!--
     Convenience wrapper for the 'ur_robot' macro which provides default values
-    for the various "parameters files" parameters for a ur30.
+    for the various "parameters files" parameters for a UR3.
     This file can be used when composing a more complex scene with one or more
-    ur30 robots.
+    UR3 robots.
     While the generic 'ur_robot' macro could also be used, it would require
     the user to provide values for all parameters, as that macro does not set
@@ -17,10 +17,10 @@
           real robot.
   -->
-  <xacro:macro name="ur30_robot" params="
+  <xacro:macro name="ur3_robot" params="
    prefix
-   joint_limits_parameters_file:='$(find ur_description)/config/ur30/joint_limits.yaml'
-   kinematics_parameters_file:='$(find ur_description)/config/ur30/default_kinematics.yaml'
-   physical_parameters_file:='$(find ur_description)/config/ur30/physical_parameters.yaml'
-   visual_parameters_file:='$(find ur_description)/config/ur30/visual_parameters.yaml'
+   joint_limits_parameters_file:='$(find ur_description)/config/ur3/joint_limits.yaml'
+   kinematics_parameters_file:='$(find ur_description)/config/ur3/default_kinematics.yaml'
+   physical_parameters_file:='$(find ur_description)/config/ur3/physical_parameters.yaml'
+   visual_parameters_file:='$(find ur_description)/config/ur3/visual_parameters.yaml'
    transmission_hw_interface:=hardware_interface/PositionJointInterface
    safety_limits:=false
@@ -28,5 +28,5 @@
    safety_k_position:=20"
   >
-    <xacro:include filename="$(find ur_description)/urdf/inc/ur_macro.xacro"/>
+    <xacro:include filename="$(find ur_description)/urdf/ur_macro.xacro"/>
     <xacro:ur_robot
       prefix="${prefix}"

File: rtb-data/rtbdata/xacro/ur_e_description/urdf/ur3e_macro.xacro (robot description, xacro)
@@ -3,7 +3,7 @@
   <!--
     Convenience wrapper for the 'ur_robot' macro which provides default values
-    for the various "parameters files" parameters for a UR16e.
+    for the various "parameters files" parameters for a UR3e.
     This file can be used when composing a more complex scene with one or more
-    UR16e robots.
+    UR3e robots.
     While the generic 'ur_robot' macro could also be used, it would require
     the user to provide values for all parameters, as that macro does not set
@@ -17,10 +17,10 @@
           real robot.
   -->
-  <xacro:macro name="ur16e_robot" params="
+  <xacro:macro name="ur3e_robot" params="
    prefix
-   joint_limits_parameters_file:='$(find ur_description)/config/ur16e/joint_limits.yaml'
-   kinematics_parameters_file:='$(find ur_description)/config/ur16e/default_kinematics.yaml'
-   physical_parameters_file:='$(find ur_description)/config/ur16e/physical_parameters.yaml'
-   visual_parameters_file:='$(find ur_description)/config/ur16e/visual_parameters.yaml'
+   joint_limits_parameters_file:='$(find ur_description)/config/ur3e/joint_limits.yaml'
+   kinematics_parameters_file:='$(find ur_description)/config/ur3e/default_kinematics.yaml'
+   physical_parameters_file:='$(find ur_description)/config/ur3e/physical_parameters.yaml'
+   visual_parameters_file:='$(find ur_description)/config/ur3e/visual_parameters.yaml'
    transmission_hw_interface:=hardware_interface/PositionJointInterface
    safety_limits:=false
@@ -28,5 +28,5 @@
    safety_k_position:=20"
   >
-    <xacro:include filename="$(find ur_description)/urdf/inc/ur_macro.xacro"/>
+    <xacro:include filename="$(find ur_description)/urdf/ur_macro.xacro"/>
     <xacro:ur_robot
       prefix="${prefix}"

File: rtb-data/rtbdata/xacro/ur_e_description/urdf/ur5_macro.xacro (robot description, xacro)
@@ -3,7 +3,7 @@
   <!--
     Convenience wrapper for the 'ur_robot' macro which provides default values
-    for the various "parameters files" parameters for a ur20.
+    for the various "parameters files" parameters for a UR5.
     This file can be used when composing a more complex scene with one or more
-    ur20 robots.
+    UR5 robots.
     While the generic 'ur_robot' macro could also be used, it would require
     the user to provide values for all parameters, as that macro does not set
@@ -17,10 +17,10 @@
           real robot.
   -->
-  <xacro:macro name="ur20_robot" params="
+  <xacro:macro name="ur5_robot" params="
    prefix
-   joint_limits_parameters_file:='$(find ur_description)/config/ur20/joint_limits.yaml'
-   kinematics_parameters_file:='$(find ur_description)/config/ur20/default_kinematics.yaml'
-   physical_parameters_file:='$(find ur_description)/config/ur20/physical_parameters.yaml'
-   visual_parameters_file:='$(find ur_description)/config/ur20/visual_parameters.yaml'
+   joint_limits_parameters_file:='$(find ur_description)/config/ur5/joint_limits.yaml'
+   kinematics_parameters_file:='$(find ur_description)/config/ur5/default_kinematics.yaml'
+   physical_parameters_file:='$(find ur_description)/config/ur5/physical_parameters.yaml'
+   visual_parameters_file:='$(find ur_description)/config/ur5/visual_parameters.yaml'
    transmission_hw_interface:=hardware_interface/PositionJointInterface
    safety_limits:=false
@@ -28,5 +28,5 @@
    safety_k_position:=20"
   >
-    <xacro:include filename="$(find ur_description)/urdf/inc/ur_macro.xacro"/>
+    <xacro:include filename="$(find ur_description)/urdf/ur_macro.xacro"/>
     <xacro:ur_robot
       prefix="${prefix}"

File: rtb-data/rtbdata/xacro/ur_e_description/urdf/ur5e_macro.xacro (robot description, xacro)
@@ -3,7 +3,7 @@
   <!--
     Convenience wrapper for the 'ur_robot' macro which provides default values
-    for the various "parameters files" parameters for a UR5.
+    for the various "parameters files" parameters for a UR5e.
     This file can be used when composing a more complex scene with one or more
-    UR5 robots.
+    UR5e robots.
     While the generic 'ur_robot' macro could also be used, it would require
     the user to provide values for all parameters, as that macro does not set
@@ -17,10 +17,10 @@
           real robot.
   -->
-  <xacro:macro name="ur5_robot" params="
+  <xacro:macro name="ur5e_robot" params="
    prefix
-   joint_limits_parameters_file:='$(find ur_description)/config/ur5/joint_limits.yaml'
-   kinematics_parameters_file:='$(find ur_description)/config/ur5/default_kinematics.yaml'
-   physical_parameters_file:='$(find ur_description)/config/ur5/physical_parameters.yaml'
-   visual_parameters_file:='$(find ur_description)/config/ur5/visual_parameters.yaml'
+   joint_limits_parameters_file:='$(find ur_description)/config/ur5e/joint_limits.yaml'
+   kinematics_parameters_file:='$(find ur_description)/config/ur5e/default_kinematics.yaml'
+   physical_parameters_file:='$(find ur_description)/config/ur5e/physical_parameters.yaml'
+   visual_parameters_file:='$(find ur_description)/config/ur5e/visual_parameters.yaml'
    transmission_hw_interface:=hardware_interface/PositionJointInterface
    safety_limits:=false
@@ -28,5 +28,5 @@
    safety_k_position:=20"
   >
-    <xacro:include filename="$(find ur_description)/urdf/inc/ur_macro.xacro"/>
+    <xacro:include filename="$(find ur_description)/urdf/ur_macro.xacro"/>
     <xacro:ur_robot
       prefix="${prefix}"

File: rtb-data/rtbdata/xacro/ur_e_description/urdf/ur_macro.xacro (robot description, xacro)
@@ -42,6 +42,6 @@
      - Muhammad Asif Rana
   -->
-  <xacro:include filename="$(find ur_description)/urdf/inc/ur_transmissions.xacro" />
-  <xacro:include filename="$(find ur_description)/urdf/inc/ur_common.xacro" />
+  <xacro:include filename="$(find ur_description)/urdf/ur_transmissions.xacro" />
+  <xacro:include filename="$(find ur_description)/urdf/ur_common.xacro" />
   <xacro:macro name="ur_robot" params="
     prefix
